File: Hackheld_Vega_PCB/Hackheld_Vega.kicad_pcb (KiCad board)
At the start: 2 copper layers, 50.5 x 67.1 mm, 35 parts, among them J1 Conn_01x04_Female, J2 Conn_01x03_Female, SW1 SW_Push, SW2 SW_Push, SW3 SW_Push, SW4 SW_Push, SW5 SW_Push, SW6 SW_Push, U1 D1_mini

Commit message: Forgotten changes
Looks like I made updates t the design without ever pushing it ¯\_(ツ)_/¯
Parts:
- moved U1 1.70 mm to (124.2, 117.2)
Connections:
- J1 pad 1: GND -> +3V3
- J1 pad 2: +3V3 -> GND
Routing:
- net GND: track 244.5 -> 241.5 mm
- net +3V3: track 20.0 -> 21.8 mm
- net /RIGHT: track 58.8 -> 60.5 mm
- net /SDA: track 30.2 -> 28.5 mm
- net /SCL: track 30.2 -> 28.5 mm
- net /B: track 36.2 -> 37.9 mm
- net /A: track 30.3 -> 32.0 mm
- net /NEOPIXEL: track 36.3 -> 38.0 mm
- net /UP: track 52.5 -> 54.1 mm
- net /DOWN: track 73.7 -> 75.4 mm
- net +5V: track 36.1 -> 36.8 mm
Other:
- board text added: "SCK"
- board text added: "VDD"
- board text removed: "3V3"
