File: Hackheld_Vega_PCB/Hackheld_Vega.sch (KiCad schematic (older format))
At the start: 10 parts, among them J1 Conn_01x04_Female, J2 Conn_01x03_Female, SW1 SW_Push, SW2 SW_Push, SW3 SW_Push, SW4 SW_Push, SW5 SW_Push, SW6 SW_Push, U1 D1_mini

Commit message: Forgotten changes
Looks like I made updates t the design without ever pushing it ¯\_(ツ)_/¯
Connections:
- net +3V3: now also J1.1 (Pin_1); no longer J1.2 (Pin_2)
- net GND: now also J1.2 (Pin_2); no longer J1.1 (Pin_1)
Changed lines of the file:
@@
 $EndComp
-Wire Wire Line
-	6300 3950 6250 3950
 Wire Wire Line
 	6300 3750 6250 3750
@@
 L power:GND #PWR011
 U 1 1 60C97073
-P 6300 4050
-F 0 "#PWR011" H 6300 3800 50  0001 C CNN
-F 1 "GND" V 6305 3922 50  0000 R CNN
-F 2 "" H 6300 4050 50  0001 C CNN
-F 3 "" H 6300 4050 50  0001 C CNN
-	1    6300 4050
-	0    -1   -1   0
+P 6400 3950
+F 0 "#PWR011" H 6400 3700 50  0001 C CNN
+F 1 "GND" H 6450 4000 50  0000 R CNN
+F 2 "" H 6400 3950 50  0001 C CNN
+F 3 "" H 6400 3950 50  0001 C CNN
+	1    6400 3950
+	1    0    0    -1
 $EndComp
 $Comp
@@
 L power:+3V3 #PWR010
 U 1 1 60C97E78
-P 6300 3950
-F 0 "#PWR010" H 6300 3800 50  0001 C CNN
-F 1 "+3V3" V 6315 4078 50  0000 L CNN
-F 2 "" H 6300 3950 50  0001 C CNN
-F 3 "" H 6300 3950 50  0001 C CNN
-	1    6300 3950
-	0    1    1    0
+P 6550 4050
+F 0 "#PWR010" H 6550 3900 50  0001 C CNN
+F 1 "+3V3" H 6450 3950 50  0000 L CNN
+F 2 "" H 6550 4050 50  0001 C CNN
+F 3 "" H 6550 4050 50  0001 C CNN
+	1    6550 4050
+	1    0    0    -1
 $EndComp
 $Comp
@@
 	1    0    0    -1
 $EndComp
+Wire Wire Line
+	6250 3950 6400 3950
+Wire Wire Line
+	6300 4050 6300 4100
+Wire Wire Line
+	6300 4100 6550 4100
+Wire Wire Line
+	6550 4100 6550 4050
 $EndSCHEMATC
