File: HackHeld Vega II/Hackheld_Vega.kicad_pcb (KiCad board)
At the start: 2 copper layers, 45.1 x 59.8 mm, 30 parts, among them J1 OLED_I2C, SW1 SW_Push, SW2 SW_Push, SW3 SW_Push, SW4 SW_Push, SW5 SW_Push, SW6 SW_Push, U1 D1_mini

Commit message: HackHeld Bat Mod PCB Files
Routing:
- added copper zone on B.Cu, net GND
- added copper zone on F.Cu, net GND
- removed copper zone on B.Cu, net (none)
- removed copper zone on F.Cu, net (none)
Other:
- board text added: "rev2"
Changed lines of the file:
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@@
     (effects (font (size 0.8 0.8) (thickness 0.16)))
+  )
+  (gr_text "rev2" (at 137.05 79.35 90) (layer "F.SilkS")
+    (effects (font (size 1.5 1.5) (thickness 0.3) bold) (justify left bottom))
   )
   (gr_text "HackHeld Vega II" (at 133.381574 98.15 90) (layer "F.SilkS")
@@
   (segment (start 153.765817 84.112) (end 154.9 82.977817) (width 0.4) (layer "F.Cu") (net 15))
   (segment (start 154.9 81) (end 153.6 79.7) (width 0.4) (layer "F.Cu") (net 15))
+  (zone (net 4) (net_name "GND") (layer "F.Cu") (hatch edge 0.508)
+    (connect_pads no (clearance 0.508))
+    (min_thickness 0.254) (filled_areas_thickness no)
+    (fill yes (mode hatch) (thermal_gap 1) (thermal_bridge_width 0.3) (smoothing chamfer) (radius 0.25) (island_removal_mode 1) (island_area_min 10)
+      (hatch_thickness 1) (hatch_gap 2) (hatch_orientation 45)
+      (hatch_border_algorithm hatch_thickness) (hatch_min_hole_area 0.3))
+    (polygon
+      (pts
+        (xy 181.35 127.35)
+        (xy 227.35 127.35)
+        (xy 227.35 64.35)
+        (xy 181.35 64.35)
+      )
+    )
+  )
   (zone (net 0) (net_name "") (layers "F&B.Cu") (hatch edge 0.508)
     (connect_pads (clearance 0))
@@
     )
   )
-  (zone (net 0) (net_name "") (layers "F&B.Cu") (hatch edge 0.508)
+  (zone (net 4) (net_name "GND") (layer "B.Cu") (hatch edge 0.508)
     (connect_pads (clearance 0.508))
     (min_thickness 0.254) (filled_areas_thickness no)
-    (fill yes (thermal_gap 1) (thermal_bridge_width 0.3) (smoothing chamfer) (radius 0.25) (island_removal_mode 1) (island_area_min 10))
+    (fill yes (mode hatch) (thermal_gap 1) (thermal_bridge_width 0.3) (smoothing chamfer) (radius 0.25)
+      (hatch_thickness 1) (hatch_gap 2) (hatch_orientation 45)
+      (hatch_border_algorithm hatch_thickness) (hatch_min_hole_area 0.3))
     (polygon
       (pts
-        (xy 129 127)
-        (xy 175 127)
-        (xy 175 64)
-        (xy 129 64)
+        (xy 181.05 127.65)
+        (xy 227.05 127.65)
+        (xy 227.05 64.65)
+        (xy 181.05 64.65)
       )
     )
